File: stlink_v3_CAN_shield.sch (EAGLE design)
At the start: 13 parts, among them CON1 STLINK_V3, U1 MCP2562-E/SN

Commit message: Update STLink footprint
Parts:
- removed C120: 1uF, rcl:C-EUC0603
- removed C126: 10n, rcl:C-EUC0603
- added C3: 100n, rcl:C-EUC0603
- added C5: 1uF, rcl:C-EUC0603
- C1: value 100n -> 1uF; OC_FARNELL 2310560 -> 2310567; OC_LOMEX 82-06-23 -> 82-07-86; OC_TME CL10B104KB8NNNC -> CL10B105KO8NNNC
- C2: value 1uF -> 10n; OC_FARNELL 2310567 -> 2310601; OC_LOMEX 82-07-86 -> 82-08-73; OC_TME CL10B105KO8NNNC -> C0603C103K1RAC
- renumbered C122 to C4, R8 to R2
Connections:
- net CAN_H renamed CAN_P
- net CAN_L renamed CAN_N
- net CAN_RX renamed CAN_MCU_N
- net CAN_TX renamed CAN_MCU_P
- net +3V3: now also C3.2, C5.1; no longer C1.2, C2.1
- net GND: now also C1.2, C3.1, C5.2; no longer C1.1, C120.2, C126.2
- net VIN_LED_R1: now also LED2.A; no longer LED1.A
- net VIN_LED_R2: now also LED1.A; no longer LED2.A
- net VUSB: now also C1.1, C2.1; no longer C120.1, C126.1
Other:
- moved on the sheet: C1, C2, LED1, LED2
